File: hardware/E106.sch (EAGLE design)
At the start: 33 parts, among them Q2 NPN, SW1 SPST_TACT-KMR2, U10 TSL2591, U11 915MHz, U5 ATMEGA328P-MU, U6 SHT35, U8 MCP1703CB, X1 16 MHz

Commit message: v1.1.0 - hardware update
- added SPI flash
- removed jumper from radio SS
- added RGB LED instead of single LED
- trace fixes
- ERC/DRC
- Silkscreen update
Parts:
- removed JP2: JUMPER-SMT_2_NC_PASTE_SILK, SparkFun-Jumpers:JUMPER-SMT_2_NC_PASTE_SILK
- removed R3: 1K, Adafruit Feather 32u4 Bluefruit LE:MICROBUILDER_RESISTOR_0402MP
- removed STAT: BLUE, microbuilder:LED0805_NOOUTLINE
- added D2: LTST-C19FD1WT, LTST-C19FD1WT:LTST-C19FD1WT
- added R1: 1K, Adafruit Feather 32u4 Bluefruit LE:MICROBUILDER_RESISTOR_0402MP
- added U1: W25X40CLUXIG_TR, W25X40CLUXIG_TR:W25X40CLUXIG_TR
Connections:
- removed net N$11: JP2.1, R7.2
- removed net N$8: R3.1, STAT.A
- new net N$6: D2.A, R1.2
- net D5: now also D2.C2
- net D6: now also D2.C3
- net D7: now also D2.C1
- net D8: now also U1.!CS
- net D9: no longer R3.2
- net GND: now also U1.EXP, U1.GND; no longer STAT.C
- net MISO: now also U1.DO(IO1)
- net MOSI: now also U1.DI(IO0)
- net SCK: now also U1.CLK
- net VCC: now also R1.1, R7.2, U1.!HOLD, U1.!WP, U1.VCC; no longer JP2.2
Other:
- note added: "1.1.0"
- note removed: "1.0.0"
- moved on the sheet: C8, CN1, J4, R2, R22, R7, R8

Commit message: minor adjustments
Changed lines of the file:
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@@
 <?xml version="1.0" encoding="utf-8"?>
 <!DOCTYPE eagle SYSTEM "eagle.dtd">
-<eagle version="9.1.1">
+<eagle version="9.5.1">
 <drawing>
 <settings>
@@
 <attribute name="VALUE" x="157.72" y="113.05" size="1.27" layer="96" font="vector" rot="R270" align="center"/>
 </instance>
-<instance part="U1" gate="G$1" x="48.26" y="40.64"/>
+<instance part="U1" gate="G$1" x="48.26" y="40.64" smashed="yes">
+<attribute name="NAME" x="40.64" y="59.055" size="1.778" layer="95"/>
+<attribute name="VALUE" x="40.64" y="22.86" size="1.778" layer="96"/>
+</instance>
 <instance part="GND6" gate="1" x="60.96" y="22.86" smashed="yes">
 <attribute name="VALUE" x="58.42" y="20.32" size="1.778" layer="96"/>
@@
 <attribute name="VALUE" x="26.924" y="54.356" size="1.778" layer="96"/>
 </instance>
-<instance part="D2" gate="G$1" x="251.46" y="-35.56" rot="R270"/>
+<instance part="D2" gate="G$1" x="251.46" y="-35.56" smashed="yes" rot="R270">
+<attribute name="NAME" x="256.547759375" y="-17.7528" size="1.271940625" layer="95" rot="R270"/>
+<attribute name="VALUE" x="254.00246875" y="-17.7627" size="1.271240625" layer="96" rot="R270"/>
+</instance>
 <instance part="SUPPLY10" gate="G$1" x="274.32" y="-30.48" smashed="yes">
 <attribute name="VALUE" x="273.304" y="-26.924" size="1.778" layer="96"/>
